File: runtime-hackpad.kicad_sch (KiCad schematic)
At the start: 4 parts, among them U1 MAX7219, U2 102010428, U3 ADXL345, U4 Buzzer

Commit message: Schematics work completed
Parts:
- added SW1: CHERRY MX, Button_Switch_Keyboard:SW_Cherry_MX_1.00u_PCB, symbol Switch:SW_Push
- added TP1: TestPoint, Connector_PinHeader_2.54mm:PinHeader_1x01_P2.54mm_Vertical, symbol Connector:TestPoint
Connections:
- net 3V3: now also TP1.1
- net GND: now also SW1.2
- net SW: now reaches U2.4 (P29/A3/D3)
- net SW: now also SW1.1
Other:
- moved on the sheet: U1, U2, U3, U4
