File: runtime-hackpad.kicad_pcb (KiCad board)
At the start: 2 copper layers, 4 parts, among them U1 MAX7219, U2 102010428, U3 ADXL345, U4 Buzzer

Commit message: Schematics work completed
Parts:
- added SW1: CHERRY MX, Button_Switch_Keyboard:SW_Cherry_MX_1.00u_PCB, F.Cu at (129.5, 93.0)
- added TP1: TestPoint, Connector_PinHeader_2.54mm:PinHeader_1x01_P2.54mm_Vertical, F.Cu at (143.3, 58.3)
- moved U3 3.98 mm to (110.0, 66.1)
- moved U1 2.84 mm to (143.5, 65.0)
- moved U4 1.86 mm to (143.5, 83.0)
Connections:
- U2 pad 4: unconnected-(U2-P29/A3/D3-Pad4) -> /SW

Commit message: PCB work
Parts:
- moved TP1 67.2 mm to (77.5, 44.5)
- moved U4 65.0 mm to (204.5, 105.5)
- moved U3 46.6 mm to (65.0, 78.1)
- moved SW1 43.0 mm to (98.1, 122.4)
- moved U2 18.2 mm to (135.5, 91.3)
- moved U1 13.2 mm to (130.9, 69.0), turned to 90 degrees
Changed lines of the file:
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@@
 	(footprint "Connector_PinHeader_2.54mm:PinHeader_1x03_P2.54mm_Vertical"
 		(layer "F.Cu")
-		(at 143.5 82.96)
+		(at 204.5 105.46)
 		(descr "Through hole straight pin header, 1x03, 2.54mm pitch, single row")
 		(tags "Through hole pin header THT 1x03 2.54mm single row")
@@
 	(footprint "Connector_PinHeader_2.54mm:PinHeader_1x08_P2.54mm_Vertical"
 		(layer "F.Cu")
-		(at 110 66.11)
+		(at 65 78.11)
 		(descr "Through hole straight pin header, 1x08, 2.54mm pitch, single row")
 		(tags "Through hole pin header THT 1x08 2.54mm single row")
@@
 	(footprint "Connector_PinHeader_2.54mm:PinHeader_1x05_P2.54mm_Vertical"
 		(layer "F.Cu")
-		(at 143.5 64.96)
+		(at 130.92 69 90)
 		(descr "Through hole straight pin header, 1x05, 2.54mm pitch, single row")
 		(tags "Through hole pin header THT 1x05 2.54mm single row")
 		(property "Reference" "U1"
-			(at 0 -2.38 0)
+			(at 0 -2.38 90)
 			(layer "F.SilkS")
 			(effects
@@
 		)
 		(property "Value" "MAX7219"
-			(at 0 12.54 0)
+			(at 0 12.54 90)
 			(layer "F.Fab")
 			(effects
@@
 		)
 		(property "Datasheet" ""
-			(at 0 0 0)
+			(at 0 0 90)
 			(layer "F.Fab")
 			(hide yes)
@@
 		)
 		(property "Description" "Generic connector, single row, 01x05, script generated"
-			(at 0 0 0)
+			(at 0 0 90)
 			(layer "F.Fab")
 			(hide yes)
@@
 		)
 		(property "KiLib_Generator" "connector/pin_header_socket"
-			(at 0 0 0)
+			(at 0 0 90)
 			(layer "F.SilkS")
 			(hide yes)
@@
 		)
 		(fp_line
+			(start 1.38 1.27)
+			(end 1.38 11.54)
+			(stroke
+				(width 0.12)
+				(type solid)
+			)
+			(layer "F.SilkS")
+		)
+		(fp_line
+			(start -1.38 1.27)
+			(end 1.38 1.27)
+			(stroke
+				(width 0.12)
+				(type solid)
+			)
+			(layer "F.SilkS")
+		)
+		(fp_line
 			(start -1.38 1.27)
 			(end -1.38 11.54)
@@
 		)
 		(fp_line
-			(start -1.38 1.27)
-			(end 1.38 1.27)
-			(stroke
-				(width 0.12)
-				(type solid)
-			)
-			(layer "F.SilkS")
-		)
-		(fp_line
 			(start -1.38 11.54)
-			(end 1.38 11.54)
-			(stroke
-				(width 0.12)
-				(type solid)
-			)
-			(layer "F.SilkS")
-		)
-		(fp_line
-			(start 1.38 1.27)
 			(end 1.38 11.54)
 			(stroke
@@
 		)
 		(fp_line
+			(start 1.27 -1.27)
+			(end 1.27 11.43)
+			(stroke
+				(width 0.1)
+				(type solid)
+			)
+			(layer "F.Fab")
+		)
+		(fp_line
+			(start -0.635 -1.27)
+			(end 1.27 -1.27)
+			(stroke
+				(width 0.1)
+				(type solid)
+			)
+			(layer "F.Fab")
+		)
+		(fp_line
 			(start -1.27 -0.635)
 			(end -0.635 -1.27)
@@
 		)
 		(fp_line
+			(start 1.27 11.43)
+			(end -1.27 11.43)
+			(stroke
+				(width 0.1)
+				(type solid)
+			)
+			(layer "F.Fab")
+		)
+		(fp_line
 			(start -1.27 11.43)
 			(end -1.27 -0.635)
@@
 			(layer "F.Fab")
 		)
-		(fp_line
-			(start -0.635 -1.27)
-			(end 1.27 -1.27)
-			(stroke
-				(width 0.1)
-				(type solid)
-			)
-			(layer "F.Fab")
-		)
-		(fp_line
-			(start 1.27 -1.27)
-			(end 1.27 11.43)
-			(stroke
-				(width 0.1)
-				(type solid)
-			)
-			(layer "F.Fab")
-		)
-		(fp_line
-			(start 1.27 11.43)
-			(end -1.27 11.43)
-			(stroke
-				(width 0.1)
-				(type solid)
-			)
-			(layer "F.Fab")
-		)
 		(fp_text user "${REFERENCE}"
-			(at 0 5.08 90)
+			(at 0 5.08 0)
 			(layer "F.Fab")
 			(effects
@@
 		)
 		(pad "1" thru_hole rect
-			(at 0 0)
+			(at 0 0 90)
 			(size 1.7 1.7)
 			(drill 1)
@@
 		)
 		(pad "2" thru_hole circle
-			(at 0 2.54)
+			(at 0 2.54 90)
 			(size 1.7 1.7)
 			(drill 1)
@@
 		)
 		(pad "3" thru_hole circle
-			(at 0 5.08)
+			(at 0 5.08 90)
 			(size 1.7 1.7)
 			(drill 1)
@@
 		)
 		(pad "4" thru_hole circle
-			(at 0 7.62)
+			(at 0 7.62 90)
 			(size 1.7 1.7)
 			(drill 1)
@@
 		)
 		(pad "5" thru_hole circle
-			(at 0 10.16)
+			(at 0 10.16 90)
 			(size 1.7 1.7)
 			(drill 1)
@@
 	(footprint "Connector_PinHeader_2.54mm:PinHeader_1x01_P2.54mm_Vertical"
 		(layer "F.Cu")
-		(at 143.295 58.295)
+		(at 77.5 44.5)
 		(descr "Through hole straight pin header, 1x01, 2.54mm pitch, single row")
 		(tags "Through hole pin header THT 1x01 2.54mm single row")
@@
 	(footprint "Seeed Studio XIAO Series Library:XIAO-RP2040-DIP"
 		(layer "F.Cu")
-		(at 127.0675 75.171 90)
+		(at 135.5 91.2685 90)
 		(property "Reference" "U2"
 			(at -0.125 -10.25 90)
@@
 	(footprint "Button_Switch_Keyboard:SW_Cherry_MX_1.00u_PCB"
 		(layer "F.Cu")
-		(at 129.5 93)
+		(at 98.12 122.42)
 		(descr "Cherry MX keyswitch, 1.00u, PCB mount, http://cherryamericas.com/wp-content/uploads/2014/12/mx_cat.pdf")
 		(tags "Cherry MX keyswitch 1.00u PCB")
@@
 		)
 	)
+	(gr_rect
+		(start 43.5 69)
+		(end 68.5 104)
+		(stroke
+			(width 0.1)
+			(type solid)
+		)
+		(fill no)
+		(layer "Dwgs.User")
+	)
+	(gr_rect
+		(start 118.54 17.5)
+		(end 155.54 72.5)
+		(stroke
+			(width 0.1)
+			(type solid)
+		)
+		(fill no)
+		(layer "Dwgs.User")
+	)
+	(gr_rect
+		(start 200 99.04)
+		(end 239 117.04)
+		(stroke
+			(width 0.1)
+			(type solid)
+		)
+		(fill no)
+		(layer "Dwgs.User")
+	)
 	(embedded_fonts no)

Commit message: pcb work done
Parts:
- moved U3 109.4 mm to (173.9, 67.5), turned to -90 degrees
- moved U4 107.5 mm to (98.5, 88.0), turned to 90 degrees
- moved TP1 65.2 mm to (117.5, 96.0)
- moved U2 57.6 mm to (165.4, 42.0)
- moved SW1 40.7 mm to (134.1, 103.4)
- moved U1 25.5 mm to (125.8, 94.0)
Routing:
- net /VCC: track 0.00 -> 148.7 mm
- net /3V3: track 0.00 -> 136.9 mm
- net /DIN: track 0.00 -> 80.8 mm, vias 0 -> 6
- net /I/O: track 0.00 -> 76.8 mm, vias 0 -> 2
- net /SW: track 0.00 -> 75.4 mm, vias 0 -> 4
- net /CS1: track 0.00 -> 72.5 mm, vias 0 -> 6
- net /CLK: track 0.00 -> 67.6 mm, vias 0 -> 6
- net /SDA: track 0.00 -> 25.2 mm
- net /SCL: track 0.00 -> 23.3 mm
- added copper zone on B.Cu, net GND
Other:
- board outline added: 91.2 x 90 mm
- board text added: "ADXL345"
- board text added: "AJ"
- board text added: "Buzzer"
- board text added: "MAX7219"
- board text added: "MX"
- board text added: "V1"
- board text added: "leveler-tool"
