File: leveler-tool.kicad_sch (KiCad schematic)
At the start: 6 parts, among them SW1 CHERRY MX, U1 MAX7219, U2 102010428, U3 ADXL345, U4 Buzzer

Commit message: header correction
Parts:
- TP1: footprint Connector_PinHeader_2.54mm:PinHeader_1x01_P2.54mm_Vertical -> Connector_PinSocket_2.54mm:PinSocket_1x01_P2.54mm_Vertical
- U1: footprint Connector_PinHeader_2.54mm:PinHeader_1x05_P2.54mm_Vertical -> Connector_PinSocket_2.54mm:PinSocket_1x05_P2.54mm_Vertical
- U3: footprint Connector_PinHeader_2.54mm:PinHeader_1x08_P2.54mm_Vertical -> Connector_PinSocket_2.54mm:PinSocket_1x08_P2.54mm_Vertical
- U4: footprint Connector_PinHeader_2.54mm:PinHeader_1x03_P2.54mm_Vertical -> Connector_PinSocket_2.54mm:PinSocket_1x03_P2.54mm_Vertical
Changed lines of the file:
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@@
 		)
 		(instances
-			(project "runtime-hackpad"
+			(project "leveler-tool"
 				(path "/b5bac4aa-c255-405e-9315-1ac9efa24788"
 					(reference "#PWR01")
@@
 		)
 		(instances
-			(project "runtime-hackpad"
+			(project "leveler-tool"
 				(path "/b5bac4aa-c255-405e-9315-1ac9efa24788"
 					(reference "#FLG03")
@@
 		)
 		(instances
-			(project "runtime-hackpad"
+			(project "leveler-tool"
 				(path "/b5bac4aa-c255-405e-9315-1ac9efa24788"
 					(reference "#PWR05")
@@
 		)
 		(instances
-			(project "runtime-hackpad"
+			(project "leveler-tool"
 				(path "/b5bac4aa-c255-405e-9315-1ac9efa24788"
 					(reference "SW1")
@@
 			)
 		)
-		(property "Footprint" "Connector_PinHeader_2.54mm:PinHeader_1x03_P2.54mm_Vertical"
+		(property "Footprint" "Connector_PinSocket_2.54mm:PinSocket_1x03_P2.54mm_Vertical"
 			(at 105.41 97.79 0)
 			(hide yes)
@@
 		)
 		(instances
-			(project "runtime-hackpad"
+			(project "leveler-tool"
 				(path "/b5bac4aa-c255-405e-9315-1ac9efa24788"
 					(reference "U4")
@@
 		)
 		(instances
-			(project "runtime-hackpad"
+			(project "leveler-tool"
 				(path "/b5bac4aa-c255-405e-9315-1ac9efa24788"
 					(reference "#PWR04")
@@
 		)
 		(instances
-			(project "runtime-hackpad"
+			(project "leveler-tool"
 				(path "/b5bac4aa-c255-405e-9315-1ac9efa24788"
 					(reference "#FLG02")
@@
 			)
 		)
-		(property "Footprint" "Connector_PinHeader_2.54mm:PinHeader_1x01_P2.54mm_Vertical"
+		(property "Footprint" "Connector_PinSocket_2.54mm:PinSocket_1x01_P2.54mm_Vertical"
 			(at 154.94 101.6 0)
 			(hide yes)
@@
 		)
 		(instances
-			(project "runtime-hackpad"
+			(project "leveler-tool"
 				(path "/b5bac4aa-c255-405e-9315-1ac9efa24788"
 					(reference "TP1")
@@
 		)
 		(instances
-			(project "runtime-hackpad"
+			(project "leveler-tool"
 				(path "/b5bac4aa-c255-405e-9315-1ac9efa24788"
 					(reference "U2")
@@
 		)
 		(instances
-			(project "runtime-hackpad"
+			(project "leveler-tool"
 				(path "/b5bac4aa-c255-405e-9315-1ac9efa24788"
 					(reference "#FLG01")
@@
 		)
 		(instances
-			(project "runtime-hackpad"
+			(project "leveler-tool"
 				(path "/b5bac4aa-c255-405e-9315-1ac9efa24788"
 					(reference "#PWR03")
@@
 		)
 		(instances
-			(project "runtime-hackpad"
+			(project "leveler-tool"
 				(path "/b5bac4aa-c255-405e-9315-1ac9efa24788"
 					(reference "#PWR02")
@@
 		)
 		(instances
-			(project "runtime-hackpad"
+			(project "leveler-tool"
 				(path "/b5bac4aa-c255-405e-9315-1ac9efa24788"
 					(reference "#PWR06")
@@
 			)
 		)
-		(property "Footprint" "Connector_PinHeader_2.54mm:PinHeader_1x05_P2.54mm_Vertical"
+		(property "Footprint" "Connector_PinSocket_2.54mm:PinSocket_1x05_P2.54mm_Vertical"
 			(at 193.04 72.39 0)
 			(hide yes)
@@
 		)
 		(instances
-			(project "runtime-hackpad"
+			(project "leveler-tool"
 				(path "/b5bac4aa-c255-405e-9315-1ac9efa24788"
 					(reference "U1")
@@
 			)
 		)
-		(property "Footprint" "Connector_PinHeader_2.54mm:PinHeader_1x08_P2.54mm_Vertical"
+		(property "Footprint" "Connector_PinSocket_2.54mm:PinSocket_1x08_P2.54mm_Vertical"
 			(at 91.44 80.01 0)
 			(hide yes)
@@
 		)
 		(instances
-			(project "runtime-hackpad"
+			(project "leveler-tool"
 				(path "/b5bac4aa-c255-405e-9315-1ac9efa24788"
 					(reference "U3")
