File: leveler-tool.kicad_pcb (KiCad board)
At the start: 2 copper layers, 91.2 x 90 mm, 6 parts, among them SW1 CHERRY MX, U1 MAX7219, U2 102010428, U3 ADXL345, U4 Buzzer

Commit message: header correction
Parts:
- added REF**: MountingHole_3.2mm_M3, MountingHole:MountingHole_3.2mm_M3, F.Cu at (174.0, 115.0)
- added REF**: MountingHole_3.2mm_M3, MountingHole:MountingHole_3.2mm_M3, F.Cu at (95.0, 115.0)
- added REF**: MountingHole_3.2mm_M3, MountingHole:MountingHole_3.2mm_M3, F.Cu at (95.0, 38.0)
- TP1: footprint Connector_PinHeader_2.54mm:PinHeader_1x01_P2.54mm_Vertical -> Connector_PinSocket_2.54mm:PinSocket_1x01_P2.54mm_Vertical
- U1: footprint Connector_PinHeader_2.54mm:PinHeader_1x05_P2.54mm_Vertical -> Connector_PinSocket_2.54mm:PinSocket_1x05_P2.54mm_Vertical
- U3: footprint Connector_PinHeader_2.54mm:PinHeader_1x08_P2.54mm_Vertical -> Connector_PinSocket_2.54mm:PinSocket_1x08_P2.54mm_Vertical
- U4: footprint Connector_PinHeader_2.54mm:PinHeader_1x03_P2.54mm_Vertical -> Connector_PinSocket_2.54mm:PinSocket_1x03_P2.54mm_Vertical
Other:
- board text added: "hackerskills"
- board text removed: "AJ"

Commit message: pcb done
Other:
- board text added: "1st"
- board text removed: "hackerskills"
Changed lines of the file:
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@@
 		)
 	)
-	(gr_text "hackerskills"
-		(at 100 116.5 0)
+	(gr_text "1st\n"
+		(at 100.4 116.5 0)
 		(layer "F.SilkS")
 		(effects
